File: Pcb-ICT-main/ict_v361-xs.brd (EAGLE design)
At the start: 18.8 x 22.8 mm, 10 parts, among them U3 Si5351, U4 ATMEGA328P-MU

Commit message: Add files via upload
Parts:
- moved C1 0.67 mm to (19.5, 25.2), turned to 270 degrees
- renumbered PU1 to R1, PU2 to R2, U$2 to GPS, U3 to U1, U4 to U2
Routing:
- net N$19: track 8.90 -> 6.80 mm, vias 1 -> 0
- net VIN: track 44.0 -> 44.9 mm
- net GND: vias 43 -> 45
- net ANT: vias 3 -> 2
Other:
- board size 18.8 x 22.8 mm -> 18.8 x 23 mm
