File: Pcb-ICT-main/ict_v361-xs.sch (EAGLE design)
At the start: 10 parts, among them U3 Si5351, U4 ATMEGA328P-MU

Commit message: Add files via upload
Parts:
- renumbered PU1 to R1, PU2 to R2, U$2 to GPS, U3 to U1, U4 to U2
